File: esp32-smart-speaker-schema/esp32-smart-speaker-schema.kicad_sch (KiCad schematic)
At the start: 19 parts, among them J1 USB_C_Receptacle_USB2.0_14P, SW1 PWR_BTN, SW2 MODE_BTN, SW3 PREV_BTN, SW4 NXT_BTN, SW5 PAUS-BTN, U2 MAX98357A

Commit message: Started developing backend for wavelet mini
Parts:
- removed SW1: PWR_BTN, symbol Switch:SW_Push_Dual
- removed SW2: MODE_BTN, symbol Switch:SW_Push_Dual
- removed SW3: PREV_BTN, symbol Switch:SW_Push_Dual
- removed SW4: NXT_BTN, symbol Switch:SW_Push_Dual
- removed SW5: PAUS-BTN, symbol Switch:SW_Push_Dual
- added SW1: PAUS_BTN, symbol Switch:SW_Push
- added SW6: PWR_BTN, symbol Switch:SW_Push
- added SW8: PREV_BTN, symbol Switch:SW_Push
- added SW9: NXT_BTN, symbol Switch:SW_Push
- renumbered D1 to DEBUG
Connections:
- net GND: now also SW1.2, SW6.2, SW8.2, SW9.2; no longer U1.1 (VIN)
- net BUZZER: now reaches BZ1.1 (+), U1.6 (GPIO27)
- net PAUS_BTN: now reaches U1.3 (GPIO13)
- net PAUS_BTN: now also SW1.1
- net BAT_LEVEL: now reaches R2.2, R3.2, U1.11 (GPIO35)
- net BAT_LEVEL: no longer RV1.2, U1.12 (GPIO34)
- net NXT_BTN: now reaches U1.24 (GPIO18)
- net NXT_BTN: now also SW9.1
- net PREV_BTN: now reaches U1.25 (GPIO19)
- net PREV_BTN: now also SW8.1
- net DIN: now reaches U1.29 (GPIO22), U2.1 (DIN)
- net PWR_BTN: now reaches U1.30 (GPIO23)
- net PWR_BTN: now also SW6.1
- net BCLK: now reaches U1.7 (GPIO26), U2.16 (BCLK)
- net LRCLK: now reaches U1.8 (GPIO25), U2.14 (LRCLK)
- new net VOLUME_POT: RV1.2, U1.12 (GPIO34)
- no-connect marks 35 -> 25
Other:
- moved on the sheet: BZ1, DEBUG, R1, RV1, U1

Commit message: Updated UI to actually display the correct manual code instead of a placeholder
Parts:
- BT1: footprint (none) -> Battery:BatteryHolder_Keystone_1042_1x18650
- BZ1: footprint (none) -> Buzzer_Beeper:Buzzer_D14mm_H7mm_P10mm
- C1: footprint (none) -> Capacitor_THT:C_Disc_D16.0mm_W5.0mm_P10.00mm
- C2: footprint (none) -> Capacitor_THT:CP_Radial_D10.0mm_P7.50mm
- DEBUG1: renamed from DEBUG; footprint (none) -> LED_THT:LED_D5.0mm
- R1, R2, R3: footprint (none) -> Resistor_THT:R_Axial_DIN0414_L11.9mm_D4.5mm_P15.24mm_Horizontal
- SW1, SW6, SW8, SW9: footprint (none) -> Button_Switch_THT:SW_PUSH_6mm
- U1: footprint ESP32_30pin -> Connector_PinSocket_2.54mm:PinSocket_1x15_P2.54mm_Vertical_SMD_Pin1Left
- U2: footprint Package_DFN_QFN:TQFN-16-1EP_3x3mm_P0.5mm_EP1.23x1.23mm -> Connector_PinHeader_1.00mm:PinHeader_1x07_P1.00mm_Vertical_SMD_Pin1Left
Changed lines of the file:
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@@
 			)
 		)
-		(property "Footprint" ""
+		(property "Footprint" "Buzzer_Beeper:Buzzer_D14mm_H7mm_P10mm"
 			(at 229.235 35.56 90)
 			(effects
@@
 			)
 		)
-		(property "Footprint" "ESP32_30pin"
+		(property "Footprint" "Connector_PinSocket_2.54mm:PinSocket_1x15_P2.54mm_Vertical_SMD_Pin1Left"
 			(at 148.59 66.04 90)
 			(effects
@@
 			)
 		)
-		(property "Footprint" ""
+		(property "Footprint" "Button_Switch_THT:SW_PUSH_6mm"
 			(at 26.67 73.66 0)
 			(effects
@@
 			)
 		)
-		(property "Footprint" ""
+		(property "Footprint" "Button_Switch_THT:SW_PUSH_6mm"
 			(at 49.53 73.66 0)
 			(effects
@@
 		(dnp no)
 		(fields_autoplaced yes)
-		(property "Reference" "DEBUG"
+		(property "Reference" "DEBUG1"
 			(at 260.0325 30.48 0)
 			(effects
@@
 			)
 		)
-		(property "Footprint" ""
+		(property "Footprint" "LED_THT:LED_D5.0mm"
 			(at 261.62 36.83 0)
 			(effects
@@
 			(project ""
 				(path "/cbac8fd8-0a29-4e40-a31e-38a1d497e26c"
-					(reference "DEBUG")
+					(reference "DEBUG1")
 					(unit 1)
 				)
@@
 			)
 		)
-		(property "Footprint" ""
+		(property "Footprint" "Capacitor_THT:C_Disc_D16.0mm_W5.0mm_P10.00mm"
 			(at 246.0752 138.43 0)
 			(effects
@@
 			)
 		)
-		(property "Footprint" "Package_DFN_QFN:TQFN-16-1EP_3x3mm_P0.5mm_EP1.23x1.23mm"
+		(property "Footprint" "Connector_PinHeader_1.00mm:PinHeader_1x07_P1.00mm_Vertical_SMD_Pin1Left"
 			(at 224.79 127 0)
 			(effects
@@
 			)
 		)
-		(property "Footprint" ""
+		(property "Footprint" "Resistor_THT:R_Axial_DIN0414_L11.9mm_D4.5mm_P15.24mm_Horizontal"
 			(at 252.222 40.64 90)
 			(effects
@@
 			)
 		)
-		(property "Footprint" ""
+		(property "Footprint" "Resistor_THT:R_Axial_DIN0414_L11.9mm_D4.5mm_P15.24mm_Horizontal"
 			(at 90.932 182.88 90)
 			(effects
@@
 			)
 		)
-		(property "Footprint" ""
+		(property "Footprint" "Capacitor_THT:CP_Radial_D10.0mm_P7.50mm"
 			(at 256.2352 138.43 0)
 			(effects
@@
 			)
 		)
-		(property "Footprint" ""
+		(property "Footprint" "Button_Switch_THT:SW_PUSH_6mm"
 			(at 93.98 73.66 0)
 			(effects
@@
 			)
 		)
-		(property "Footprint" ""
+		(property "Footprint" "Battery:BatteryHolder_Keystone_1042_1x18650"
 			(at 85.344 173.99 90)
 			(effects
@@
 			)
 		)
-		(property "Footprint" ""
+		(property "Footprint" "Resistor_THT:R_Axial_DIN0414_L11.9mm_D4.5mm_P15.24mm_Horizontal"
 			(at 73.152 182.88 90)
 			(effects
@@
 			)
 		)
-		(property "Footprint" ""
+		(property "Footprint" "Button_Switch_THT:SW_PUSH_6mm"
 			(at 71.12 73.66 0)
 			(effects
