File: esp32-smart-speaker-schema/wavelet_mini.kicad_sch (KiCad schematic)
At the start: 0 parts

Commit message: Started developing backend for wavelet mini
Parts:
- added BT1: Battery, symbol Device:Battery
- added BZ1: Buzzer, symbol Device:Buzzer
- added C1: 100n, symbol Device:C
- added ESP32-S3 Display Module: ~, symbol added_by_me:ESP32_S3_Display_Module
- added LS1: Speaker, symbol Device:Speaker
- added PWR_BTN, VOL_BTN+, VOL_BTN-: SW_Push, symbol Switch:SW_Push
- added R1: LDR03, OptoDevice:R_LDR_10x8.5mm_P7.6mm_Vertical, symbol Sensor_Optical:LDR03
- added R4: 10k, symbol Device:R
Connections:
- new net: BT1.1 (+), ESP32-S3 Display Module. (IO2)
- new net: BT1.2 (-), ESP32-S3 Display Module. (IO2)
- new net: ESP32-S3 Display Module. (IO2), LS1.1
- new net: ESP32-S3 Display Module. (IO2), LS1.2
- new net 3.3V: C1.1, ESP32-S3 Display Module. (IO2), R1.2
- new net GND: BZ1.2 (-), C1.2, ESP32-S3 Display Module. (IO2), PWR_BTN.2, R4.1, VOL_BTN+.2, VOL_BTN-.2
- new net GPIO14: ESP32-S3 Display Module. (IO2), PWR_BTN.1
- new net GPIO15: ESP32-S3 Display Module. (IO2), VOL_BTN-.1
- new net GPIO16: ESP32-S3 Display Module. (IO2), VOL_BTN+.1
- new net GPIO2: BZ1.1 (+), ESP32-S3 Display Module. (IO2)
- new net GPIO3: ESP32-S3 Display Module. (IO2), R1.1, R4.2

Commit message: Finally started development for Wavelet Mini.
What's new:
- QR code onboarding
- Touchscreen drivers
- EEZ Studio UI integration
- Firmware refactor for Mini
- ESP32-S3 compatibility

Regression:
- Wavelet Regular is no longer feeling very regular.
Parts:
- ESP32-S3 Display Module1: renamed from ESP32-S3 Display Module
- renumbered PWR_BTN to PWR_BTN1, VOL_BTN+ to VOL_BTN+1, VOL_BTN- to VOL_BTN-1
Connections:
- no-connect marks 0 -> 3
Other:
- title: Wavelet Speaker -> Wavelet Mini
Changed lines of the file:
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@@
 	(paper "A4")
 	(title_block
-		(title "Wavelet Speaker")
+		(title "Wavelet Mini")
 		(date "2026-03-12")
 		(rev "1.0.0")
@@
 		(diameter 0)
 		(color 0 0 0 0)
+	)
+	(no_connect
+		(at 83.82 90.17)
+	)
+	(no_connect
+		(at 78.74 90.17)
+	)
+	(no_connect
+		(at 86.36 90.17)
 	)
 	(wire
@@
 		(dnp no)
 		(fields_autoplaced yes)
-		(property "Reference" "VOL_BTN-?"
+		(property "Reference" "VOL_BTN-1"
 			(at 166.37 52.07 0)
 			(effects
@@
 			(project "wavelet_mini"
 				(path "/0c3772f6-de72-4c77-9f16-5e9ca2dd1615"
-					(reference "VOL_BTN-")
+					(reference "VOL_BTN-1")
 					(unit 1)
 				)
@@
 		(dnp no)
 		(fields_autoplaced yes)
-		(property "Reference" "PWR_BTN?"
+		(property "Reference" "PWR_BTN1"
 			(at 109.22 52.07 0)
 			(effects
@@
 			(project ""
 				(path "/0c3772f6-de72-4c77-9f16-5e9ca2dd1615"
-					(reference "PWR_BTN")
+					(reference "PWR_BTN1")
 					(unit 1)
 				)
@@
 		(dnp no)
 		(fields_autoplaced yes)
-		(property "Reference" "BT?"
+		(property "Reference" "BT1"
 			(at 67.8815 97.79 90)
 			(effects
@@
 		(dnp no)
 		(fields_autoplaced yes)
-		(property "Reference" "ESP32-S3 Display Module?"
+		(property "Reference" "ESP32-S3 Display Module1"
 			(at 97.79 78.8669 0)
 			(effects
@@
 			(project ""
 				(path "/0c3772f6-de72-4c77-9f16-5e9ca2dd1615"
-					(reference "ESP32-S3 Display Module")
+					(reference "ESP32-S3 Display Module1")
 					(unit 1)
 				)
@@
 		(on_board yes)
 		(dnp no)
-		(property "Reference" "LS?"
+		(property "Reference" "LS1"
 			(at 50.038 56.896 90)
 			(effects
@@
 		(dnp no)
 		(fields_autoplaced yes)
-		(property "Reference" "R?"
+		(property "Reference" "R4"
 			(at 149.86 91.44 90)
 			(effects
@@
 		(dnp no)
 		(fields_autoplaced yes)
-		(property "Reference" "R?"
+		(property "Reference" "R1"
 			(at 130.81 88.9 90)
 			(effects
@@
 		(dnp no)
 		(fields_autoplaced yes)
-		(property "Reference" "BZ?"
+		(property "Reference" "BZ1"
 			(at 171.45 76.1999 0)
 			(effects
@@
 		(dnp no)
 		(fields_autoplaced yes)
-		(property "Reference" "#PWR?"
+		(property "Reference" "#PWR01"
 			(at 114.3 66.04 0)
 			(effects
@@
 		(dnp no)
 		(fields_autoplaced yes)
-		(property "Reference" "VOL_BTN+?"
+		(property "Reference" "VOL_BTN+1"
 			(at 134.62 52.07 0)
 			(effects
@@
 			(project "wavelet_mini"
 				(path "/0c3772f6-de72-4c77-9f16-5e9ca2dd1615"
-					(reference "VOL_BTN+")
+					(reference "VOL_BTN+1")
 					(unit 1)
 				)
@@
 		(dnp no)
 		(fields_autoplaced yes)
-		(property "Reference" "#PWR?"
+		(property "Reference" "#PWR02"
 			(at 85.09 62.23 0)
 			(effects
@@
 		(dnp no)
 		(fields_autoplaced yes)
-		(property "Reference" "#PWR?"
+		(property "Reference" "#PWR05"
 			(at 160.02 104.14 0)
 			(effects
@@
 		(dnp no)
 		(fields_autoplaced yes)
-		(property "Reference" "C?"
+		(property "Reference" "C1"
 			(at 85.09 36.8299 0)
 			(effects
@@
 		(dnp no)
 		(fields_autoplaced yes)
-		(property "Reference" "#PWR?"
+		(property "Reference" "#PWR07"
 			(at 81.28 96.52 0)
 			(effects
@@
 		(dnp no)
 		(fields_autoplaced yes)
-		(property "Reference" "#PWR?"
+		(property "Reference" "#PWR03"
 			(at 139.7 66.04 0)
 			(effects
@@
 		(dnp no)
 		(fields_autoplaced yes)
-		(property "Reference" "#PWR?"
+		(property "Reference" "#PWR08"
 			(at 78.74 63.5 0)
 			(effects
@@
 		(dnp no)
 		(fields_autoplaced yes)
-		(property "Reference" "#PWR?"
+		(property "Reference" "#PWR06"
 			(at 165.1 86.36 0)
 			(effects
@@
 		(dnp no)
 		(fields_autoplaced yes)
-		(property "Reference" "#PWR?"
+		(property "Reference" "#PWR09"
 			(at 81.28 48.26 0)
 			(effects
@@
 		(dnp no)
 		(fields_autoplaced yes)
-		(property "Reference" "#PWR?"
+		(property "Reference" "#PWR04"
 			(at 171.45 66.04 0)
 			(effects

Commit message: Updated UI to actually display the correct manual code instead of a placeholder
Parts:
- BT2: renamed from BT1; footprint (none) -> Battery:BatteryHolder_Keystone_1042_1x18650
- BZ2: renamed from BZ1; footprint (none) -> Buzzer_Beeper:Buzzer_D14mm_H7mm_P10mm
- C3: renamed from C1; footprint (none) -> Capacitor_THT:C_Disc_D16.0mm_W5.0mm_P10.00mm
- PWR_BTN1, VOL_BTN+1, VOL_BTN-1: footprint (none) -> Button_Switch_THT:SW_PUSH_6mm
- R5: renamed from R4; footprint (none) -> Resistor_THT:R_Axial_DIN0414_L11.9mm_D4.5mm_P15.24mm_Horizontal
- renumbered LS1 to LS2, R1 to R4
Changed lines of the file:
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@@
 			)
 		)
-		(property "Footprint" ""
+		(property "Footprint" "Button_Switch_THT:SW_PUSH_6mm"
 			(at 166.37 54.61 0)
 			(effects
@@
 			(project "esp32-smart-speaker-schema"
 				(path "/cbac8fd8-0a29-4e40-a31e-38a1d497e26c/4025826d-41bd-4ce8-a151-2a14cf6b28c1"
-					(reference "VOL_BTN-?")
+					(reference "VOL_BTN-1")
 					(unit 1)
 				)
@@
 			)
 		)
-		(property "Footprint" ""
+		(property "Footprint" "Button_Switch_THT:SW_PUSH_6mm"
 			(at 109.22 54.61 0)
 			(effects
@@
 			(project "esp32-smart-speaker-schema"
 				(path "/cbac8fd8-0a29-4e40-a31e-38a1d497e26c/4025826d-41bd-4ce8-a151-2a14cf6b28c1"
-					(reference "PWR_BTN?")
+					(reference "PWR_BTN1")
 					(unit 1)
 				)
@@
 		(dnp no)
 		(fields_autoplaced yes)
-		(property "Reference" "BT1"
+		(property "Reference" "BT2"
 			(at 67.8815 97.79 90)
 			(effects
@@
 			)
 		)
-		(property "Footprint" ""
+		(property "Footprint" "Battery:BatteryHolder_Keystone_1042_1x18650"
 			(at 68.834 105.41 90)
 			(effects
@@
 			(project "esp32-smart-speaker-schema"
 				(path "/cbac8fd8-0a29-4e40-a31e-38a1d497e26c/4025826d-41bd-4ce8-a151-2a14cf6b28c1"
-					(reference "BT?")
+					(reference "BT2")
 					(unit 1)
 				)
@@
 			(project "esp32-smart-speaker-schema"
 				(path "/cbac8fd8-0a29-4e40-a31e-38a1d497e26c/4025826d-41bd-4ce8-a151-2a14cf6b28c1"
-					(reference "ESP32-S3 Display Module?")
+					(reference "ESP32-S3 Display Module1")
 					(unit 1)
 				)
@@
 		(on_board yes)
 		(dnp no)
-		(property "Reference" "LS1"
+		(property "Reference" "LS2"
 			(at 50.038 56.896 90)
 			(effects
@@
 			(project "esp32-smart-speaker-schema"
 				(path "/cbac8fd8-0a29-4e40-a31e-38a1d497e26c/4025826d-41bd-4ce8-a151-2a14cf6b28c1"
-					(reference "LS?")
+					(reference "LS2")
 					(unit 1)
 				)
@@
 		(dnp no)
 		(fields_autoplaced yes)
-		(property "Reference" "R4"
+		(property "Reference" "R5"
 			(at 149.86 91.44 90)
 			(effects
@@
 			)
 		)
-		(property "Footprint" ""
+		(property "Footprint" "Resistor_THT:R_Axial_DIN0414_L11.9mm_D4.5mm_P15.24mm_Horizontal"
 			(at 149.86 96.012 90)
 			(effects
@@
 			(project "esp32-smart-speaker-schema"
 				(path "/cbac8fd8-0a29-4e40-a31e-38a1d497e26c/4025826d-41bd-4ce8-a151-2a14cf6b28c1"
-					(reference "R?")
+					(reference "R5")
 					(unit 1)
 				)
@@
 		(dnp no)
 		(fields_autoplaced yes)
-		(property "Reference" "R1"
+		(property "Reference" "R4"
 			(at 130.81 88.9 90)
 			(effects
@@
 			(project "esp32-smart-speaker-schema"
 				(path "/cbac8fd8-0a29-4e40-a31e-38a1d497e26c/4025826d-41bd-4ce8-a151-2a14cf6b28c1"
-					(reference "R?")
+					(reference "R4")
 					(unit 1)
 				)
@@
 		(dnp no)
 		(fields_autoplaced yes)
-		(property "Reference" "BZ1"
+		(property "Reference" "BZ2"
 			(at 171.45 76.1999 0)
 			(effects
@@
 			)
 		)
-		(property "Footprint" ""
+		(property "Footprint" "Buzzer_Beeper:Buzzer_D14mm_H7mm_P10mm"
 			(at 167.005 74.93 90)
 			(effects
@@
 			(project "esp32-smart-speaker-schema"
 				(path "/cbac8fd8-0a29-4e40-a31e-38a1d497e26c/4025826d-41bd-4ce8-a151-2a14cf6b28c1"
-					(reference "BZ?")
+					(reference "BZ2")
 					(unit 1)
 				)
@@
 		(dnp no)
 		(fields_autoplaced yes)
-		(property "Reference" "#PWR01"
+		(property "Reference" "#PWR0109"
 			(at 114.3 66.04 0)
 			(effects
@@
 			(project "esp32-smart-speaker-schema"
 				(path "/cbac8fd8-0a29-4e40-a31e-38a1d497e26c/4025826d-41bd-4ce8-a151-2a14cf6b28c1"
-					(reference "#PWR?")
+					(reference "#PWR0109")
 					(unit 1)
 				)
@@
 			)
 		)
-		(property "Footprint" ""
+		(property "Footprint" "Button_Switch_THT:SW_PUSH_6mm"
 			(at 134.62 54.61 0)
 			(effects
@@
 			(project "esp32-smart-speaker-schema"
 				(path "/cbac8fd8-0a29-4e40-a31e-38a1d497e26c/4025826d-41bd-4ce8-a151-2a14cf6b28c1"
-					(reference "VOL_BTN+?")
+					(reference "VOL_BTN+1")
 					(unit 1)
 				)
@@
 		(dnp no)
 		(fields_autoplaced yes)
-		(property "Reference" "#PWR02"
+		(property "Reference" "#PWR0104"
 			(at 85.09 62.23 0)
 			(effects
@@
 			(project "esp32-smart-speaker-schema"
 				(path "/cbac8fd8-0a29-4e40-a31e-38a1d497e26c/4025826d-41bd-4ce8-a151-2a14cf6b28c1"
-					(reference "#PWR?")
+					(reference "#PWR0104")
 					(unit 1)
 				)
@@
 		(dnp no)
 		(fields_autoplaced yes)
-		(property "Reference" "#PWR05"
+		(property "Reference" "#PWR0106"
 			(at 160.02 104.14 0)
 			(effects
@@
 			(project "esp32-smart-speaker-schema"
 				(path "/cbac8fd8-0a29-4e40-a31e-38a1d497e26c/4025826d-41bd-4ce8-a151-2a14cf6b28c1"
-					(reference "#PWR?")
+					(reference "#PWR0106")
 					(unit 1)
 				)
@@
 		(dnp no)
 		(fields_autoplaced yes)
-		(property "Reference" "C1"
+		(property "Reference" "C3"
 			(at 85.09 36.8299 0)
 			(effects
@@
 			)
 		)
-		(property "Footprint" ""
+		(property "Footprint" "Capacitor_THT:C_Disc_D16.0mm_W5.0mm_P10.00mm"
 			(at 82.2452 41.91 0)
 			(effects
@@
 			(project "esp32-smart-speaker-schema"
 				(path "/cbac8fd8-0a29-4e40-a31e-38a1d497e26c/4025826d-41bd-4ce8-a151-2a14cf6b28c1"
-					(reference "C?")
+					(reference "C3")
 					(unit 1)
 				)
@@
 		(dnp no)
 		(fields_autoplaced yes)
-		(property "Reference" "#PWR07"
+		(property "Reference" "#PWR0101"
 			(at 81.28 96.52 0)
 			(effects
@@
 			(project "esp32-smart-speaker-schema"
 				(path "/cbac8fd8-0a29-4e40-a31e-38a1d497e26c/4025826d-41bd-4ce8-a151-2a14cf6b28c1"
-					(reference "#PWR?")
+					(reference "#PWR0101")
 					(unit 1)
 				)
@@
 		(dnp no)
 		(fields_autoplaced yes)
-		(property "Reference" "#PWR03"
+		(property "Reference" "#PWR0105"
 			(at 139.7 66.04 0)
 			(effects
@@
 			(project "esp32-smart-speaker-schema"
 				(path "/cbac8fd8-0a29-4e40-a31e-38a1d497e26c/4025826d-41bd-4ce8-a151-2a14cf6b28c1"
-					(reference "#PWR?")
+					(reference "#PWR0105")
 					(unit 1)
 				)
@@
 		(dnp no)
 		(fields_autoplaced yes)
-		(property "Reference" "#PWR08"
+		(property "Reference" "#PWR0102"
 			(at 78.74 63.5 0)
 			(effects
@@
 			(project "esp32-smart-speaker-schema"
 				(path "/cbac8fd8-0a29-4e40-a31e-38a1d497e26c/4025826d-41bd-4ce8-a151-2a14cf6b28c1"
-					(reference "#PWR?")
+					(reference "#PWR0102")
 					(unit 1)
 				)
@@
 		(dnp no)
 		(fields_autoplaced yes)
-		(property "Reference" "#PWR06"
+		(property "Reference" "#PWR0107"
 			(at 165.1 86.36 0)
 			(effects
@@
 			(project "esp32-smart-speaker-schema"
 				(path "/cbac8fd8-0a29-4e40-a31e-38a1d497e26c/4025826d-41bd-4ce8-a151-2a14cf6b28c1"
-					(reference "#PWR?")
+					(reference "#PWR0107")
 					(unit 1)
 				)
@@
 		(dnp no)
 		(fields_autoplaced yes)
-		(property "Reference" "#PWR09"
+		(property "Reference" "#PWR0103"
 			(at 81.28 48.26 0)
 			(effects
@@
 			(project "esp32-smart-speaker-schema"
 				(path "/cbac8fd8-0a29-4e40-a31e-38a1d497e26c/4025826d-41bd-4ce8-a151-2a14cf6b28c1"
-					(reference "#PWR?")
+					(reference "#PWR0103")
 					(unit 1)
 				)
@@
 		(dnp no)
 		(fields_autoplaced yes)
-		(property "Reference" "#PWR04"
+		(property "Reference" "#PWR0108"
 			(at 171.45 66.04 0)
 			(effects
@@
 			(project "esp32-smart-speaker-schema"
 				(path "/cbac8fd8-0a29-4e40-a31e-38a1d497e26c/4025826d-41bd-4ce8-a151-2a14cf6b28c1"
-					(reference "#PWR?")
-					(unit 1)
-				)
+					(reference "#PWR0108")
+					(unit 1)
+				)
